File: AntHat.kicad_sch (KiCad schematic)
At the start: 66 parts, among them J1 Raspberry_Pi_2_3, J2 0455580003, J3 PSU Comm, J4 61900411021, J5 61900411021, J6 0353180420, J7 0353180420, Q1 DMP3013SFV-7, U1 AP64501SP-13, U2 EMC2305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

Commit message: added fiducials
Parts:
- added FID1, FID2, FID3, FID4: Fiducial, Fiducial:Fiducial_0.5mm_Mask1mm, symbol Mechanical:Fiducial

Commit message: add BOM add iBOM
Parts:
- C21: LCSC C107021 -> C16529
- G2: now left out of the parts list
Changed lines of the file:
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@@
 			)
 		)
-		(property "LCSC" "C107021"
+		(property "LCSC" "C16529"
 			(at 306.07 63.5 0)
 			(effects
@@
 		(unit 1)
 		(exclude_from_sim no)
-		(in_bom yes)
+		(in_bom no)
 		(on_board yes)
 		(dnp no)
